File: LiDAR_Lite_Interface_CAN.brd (EAGLE design)
At the start: 50.2 x 56.2 mm, 30 parts, among them J1 CONN_6SCREW_2.54, J2 CONN_42.54_SCREW, Q1 2N7002, Q2 2N7002, Q3 DMG3404, Q4 MOSFET_PCH-NX2301P, U1 TLV61220DBV, U2 TS5A23157DGS

Commit message: Updated layout, added variants
Improved layout, potentially add button, then ready to send to fab. Added variations of layout for potential future alteration
Parts:
- XTAL1: value CRYSTAL_SHIELD3.2X2.5 -> CRYSTALHC-49/US; device bschulz:CRYSTAL_3.2X2.5_4-SMD -> bschulz:HC49UP
- moved XTAL1 56.9 mm to (7.62, -3.81), turned to 0 degrees
Connections:
- net GND: no longer XTAL1.2, XTAL1.4
- net N$1: now also XTAL1.2; no longer XTAL1.3
Routing:
- net GND: track 128.8 -> 126.6 mm
- net N$1: track 6.99 -> 6.26 mm
Changed lines of the file:
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@@
 <drawing>
 <settings>
-<setting alwaysvectorfont="yes"/>
+<setting alwaysvectorfont="no"/>
 <setting verticaltext="up"/>
 </settings>
@@
 <attribute name="VALUE" x="16.51" y="21.971" size="0.6096" layer="27" font="vector" ratio="20" rot="R180" align="top-center"/>
 </element>
-<element name="XTAL1" library="bschulz" package="CRYSTAL_3.2X2.5_4-SMD" value="CRYSTAL_SHIELD3.2X2.5" x="24.13" y="50.673" smashed="yes" rot="R270">
-<attribute name="DIGIKEY" value="535-10901-1-ND" x="24.13" y="50.673" size="1.778" layer="27" rot="R270" display="off"/>
-<attribute name="MF" value="Abricon" x="24.13" y="50.673" size="1.778" layer="27" rot="R270" display="off"/>
-<attribute name="MPN" value="ABM8G-12.000MHZ-4Y-T3" x="24.13" y="50.673" size="1.778" layer="27" rot="R270" display="off"/>
-<attribute name="NAME" x="26.162" y="50.673" size="0.6096" layer="25" font="vector" ratio="15" rot="R270" align="center"/>
-</element>
 <element name="C2" library="bschulz_passives" package="C0603" value="" x="20.828" y="51.816" smashed="yes">
 <attribute name="DIGIKEY" value="311-1058-1-ND" x="20.828" y="51.816" size="1.778" layer="27" display="off"/>
@@
 <attribute name="MPN" value="TS5A23157DGSR" x="29.337" y="33.274" size="1.778" layer="27" rot="R270" display="off"/>
 <attribute name="NAME" x="27.178" y="33.274" size="0.6096" layer="25" font="vector" ratio="15" rot="R270" align="center"/>
+</element>
+<element name="XTAL1" library="bschulz" package="HC49UP" value="CRYSTALHC-49/US" x="7.62" y="-3.81" smashed="yes">
+<attribute name="NAME" x="7.366" y="-1.143" size="0.6096" layer="25" font="vector" ratio="20" align="bottom-center"/>
+<attribute name="VALUE" x="7.62" y="-6.477" size="0.6096" layer="27" font="vector" ratio="20" align="top-center"/>
 </element>
 </elements>
@@
 <contactref element="D1" pad="CATHODE"/>
 <contactref element="U2" pad="3"/>
-<contactref element="C5" pad="1"/>
-<contactref element="XTAL1" pad="2"/>
-<contactref element="XTAL1" pad="4"/>
-<contactref element="C2" pad="1"/>
 <wire x1="31.75" y1="12.78" x2="31.75" y2="11.938" width="0.4064" layer="1"/>
 <wire x1="32.07" y1="11.618" x2="34.417" y2="11.618" width="0.4064" layer="1"/>
@@
 <vertex x="19.558" y="52.959"/>
 <vertex x="25.654" y="52.959"/>
-<vertex x="25.654" y="52.959"/>
 <vertex x="26.035" y="52.578"/>
 <vertex x="26.035" y="48.641"/>
@@
 <vertex x="19.05" y="48.895"/>
 </polygon>
-<wire x1="19.978" y1="50.673" x2="19.978" y2="49.657" width="0.254" layer="1"/>
 <via x="19.978" y="50.673" extent="1-16" drill="0.254"/>
-<wire x1="19.978" y1="51.816" x2="19.978" y2="50.673" width="0.254" layer="1"/>
 <wire x1="16.51" y1="47.752" x2="19.431" y2="50.673" width="0.4064" layer="16"/>
 <wire x1="19.431" y1="50.673" x2="19.978" y2="50.673" width="0.4064" layer="16"/>
@@
 <wire x1="21.717" y1="37.465" x2="27.127028125" y2="32.054971875" width="0.3048" layer="1"/>
 <via x="27.127028125" y="32.054971875" extent="1-16" drill="0.254"/>
+<contactref element="C2" pad="1"/>
+<contactref element="C5" pad="1"/>
 </signal>
 <signal name="5V_SW">
@@
 </signal>
 <signal name="N$1">
-<contactref element="XTAL1" pad="3"/>
 <contactref element="C5" pad="2"/>
 <contactref element="U3" pad="13"/>
-<wire x1="24.93" y1="49.573" x2="25.395" y2="50.038" width="0.254" layer="1"/>
 <wire x1="25.395" y1="50.038" x2="27.531" y2="50.038" width="0.254" layer="1"/>
-<wire x1="24.93" y1="49.573" x2="24.93" y2="49.50286875" width="0.254" layer="1"/>
 <wire x1="24.93" y1="49.50286875" x2="24.02073125" y2="48.5936" width="0.254" layer="1"/>
 <wire x1="22.63926875" y1="48.5936" x2="21.678" y2="49.55486875" width="0.254" layer="1"/>
 <wire x1="21.678" y1="49.55486875" x2="21.678" y2="49.657" width="0.254" layer="1"/>
 <wire x1="24.02073125" y1="48.5936" x2="22.63926875" y2="48.5936" width="0.254" layer="1"/>
+<contactref element="XTAL1" pad="2"/>
+<wire x1="24.93" y1="49.50286875" x2="25.395" y2="50.038" width="0" layer="19" extent="1-1"/>
+<wire x1="12.446" y1="-3.81" x2="22.63926875" y2="48.5936" width="0" layer="19" extent="1-1"/>
 </signal>
 <signal name="N$3">
 <contactref element="C2" pad="2"/>
-<contactref element="XTAL1" pad="1"/>
 <contactref element="U3" pad="12"/>
 <wire x1="27.531" y1="51.308" x2="26.13513125" y2="51.308" width="0.254" layer="1"/>
@@
 <wire x1="25.62073125" y1="50.7936" x2="24.11226875" y2="50.7936" width="0.254" layer="1"/>
 <wire x1="24.11226875" y1="50.7936" x2="23.33" y2="51.575875" width="0.254" layer="1"/>
-<wire x1="23.33" y1="51.575875" x2="23.33" y2="51.773" width="0.254" layer="1"/>
 <wire x1="21.678" y1="51.816" x2="23.287" y2="51.816" width="0.254" layer="1"/>
-<wire x1="23.287" y1="51.816" x2="23.33" y2="51.773" width="0.254" layer="1"/>
+<contactref element="XTAL1" pad="1"/>
+<wire x1="23.287" y1="51.816" x2="23.33" y2="51.575875" width="0" layer="19" extent="1-1"/>
+<wire x1="2.794" y1="-3.81" x2="24.11226875" y2="50.7936" width="0" layer="19" extent="1-1"/>
 </signal>
 <signal name="MISO">
@@
 </board>
 </drawing>
+<compatibility>
+<note version="8.3" severity="warning">
+Since Version 8.3, EAGLE supports URNs for individual library
+assets (packages, symbols, and devices). The URNs of those assets
+will not be understood (or retained) with this version.
+</note>
+</compatibility>
 </eagle>
